Commit message: change laser floor fow and add vsmu in vehicle execution node

File: gazebo_oru/cititruck/cititruck_description/urdf/cititruck.xacro (robot description, xacro)
@@ -42,5 +42,5 @@
         <box size="0.4 0.55 0.75" />
       </geometry>
-      <material name="red"/>
+      <material name="blue"/>
     </visual>
     <collision>
